File: pcb/micro-board.sch (EAGLE design)
At the start: 7 parts, among them IC1 STM32F401RET6U, IC2 LDS3985M33R

Commit message: Updated the PCB Schematic: 80% complete. Added PCB reference.
Parts:
- added C10, C14, C15, C7, C9: 0.1uF, LinnesLab-Passives:CAPACITOR0603
- added C11, C8: 1uF, LinnesLab-Passives:CAPACITOR0603
- added C12, C18: 10nF, LinnesLab-Passives:CAPACITOR0603
- added C13, C16, C17, C6: 10uF, LinnesLab-Passives:CAPACITOR0603
- added IC3: LDS3985M33R, SamacSys_Parts:LDS3985M33R
- added IC4: HX711, SamacSys_Parts:HX711
- added J1, J2: (no value), LinnesLab-Connectors:CONN_03
- added J10, J6: (no value), LinnesLab-Connectors:CONN_05
- added J11, J3, J5, J7, J8: (no value), LinnesLab-Connectors:CONN_04
- added J4, J9: (no value), LinnesLab-Connectors:CONN_02
- added Q1: S8550, SamacSys_Parts:S8550
- added R1, R2: 100k, LinnesLab-Passives:RESISTOR0603
- added R10, R11, R14, R5, R6, R9: 10k, LinnesLab-Passives:RESISTOR0603
- added R12: 47k, LinnesLab-Passives:RESISTOR0603
- added R13: 1k, LinnesLab-Passives:RESISTOR0603
- added R3: 8.2k, LinnesLab-Passives:RESISTOR0603
- added R4: 6.8k, LinnesLab-Passives:RESISTOR0603
- added S1: MOMENTARY-SWITCH-SPST-SMD-5.2-REDUNDANT, SparkFun-Switches:MOMENTARY-SWITCH-SPST-SMD-5.2-REDUNDANT
- added SJ1: 3V3 Jumper, jumper:SJ
- added SJ2: GND Jumper, jumper:SJ
- added SV1, SV2: (no value), con-lsta:FE20-1
- added U$1: PAD, LinnesLab-Connectors:PAD
Connections:
- net N$1 renamed VDD
- new net 3.3V: C13.1, C14.1, C15.1, C16.1, IC1.VBAT, IC1.VDD_1, IC1.VDD_2, IC1.VDD_3, IC1.VDD_4, IC4.DVDD, IC4.VSUP, J5.4, J6.5, J8.4, J9.1, J9.2, Q1.E, R1.2, R10.2, R11.2, R12.1, R14.2, R9.2, SJ1.2, SV1.19, SV2.19
- new net AVDD: IC4.AVDD, J7.4, Q1.C, R3.2
- new net CH+: IC4.INNA, IC4.INPB, J7.2
- new net CH-: IC4.INNB, IC4.INPA, J7.1
- new net D0: SV1.8
- new net D1: SV1.7
- new net D2: SV1.6
- new net D3: SV1.5
- new net D4: SV1.4
- new net D5: SV1.3
- new net D6: SV1.2
- new net D7: SV1.1
- new net HSE_IN: IC1.PH0-_OSC_IN
- new net HSE_OUT: IC1.PH1-_OSC_OUT
- new net HX_CLK: IC1.PB9, J8.1
- new net HX_CLOCK: IC4.PD_SCK, J5.1
- new net HX_DATA: IC1.PB8, J8.2
- new net HX_SDA: IC4.DOUT, J5.2
- new net IM0: R5.2, SV2.3
- new net IM1: R6.2, SV2.4
- new net LITE: IC1.PC8, R14.1, SV1.13, SV2.11, U$1.1
- new net MEM_SCL: IC1.PB6
- new net MEM_SDA: IC1.PB7
- new net N$1: C9.2, IC3.BYPASS
- new net N$11: C17.2, IC4.VBG
- new net N$12: IC4.RATE, SJ1.1, SJ2.1
- new net N$15: IC1.BOOT0, R11.1
- new net N$17: R13.1, S1.2
- new net N$19: C18.2, R13.2
- new net N$31: SV2.18
- new net N$8: C11.1, C12.1, IC1.VCAP1
- new net NRST: C18.1, IC1.NRST, R12.2, S1.1
- new net OLED_MOSI: IC1.PC12
- new net OLED_NSS: IC1.PC11
- new net OLED_SCK: IC1.PC10
- new net PA10: IC1.PA10, J1.3
- new net PA11: IC1.PA11, J1.2
- new net PA12: IC1.PA12, J1.1
- new net PB3: IC1.PB3, J2.3
- new net PB4: IC1.PB4, J2.2
- new net PB5: IC1.PB5, J2.1
- new net PC0: IC1.PC0, J3.4
- new net PC1: IC1.PC1, J3.3
- new net PC2: IC1.PC2, J3.2
- new net PC3: IC1.PC3, J3.1
- new net RD: SV1.15
- new net SD_CS: IC1.PC9, R9.1, SV2.2
- new net SD_DC: IC1.PA8
- new net SD_DET: IC1.PA9, SV2.1
- new net SS_CS: IC1.PA4, J6.2
- new net SS_MISO: IC1.PA6
- new net SS_MOSI: IC1.PA7, J6.3
- new net SS_SCK: IC1.PA5, J6.1
- new net SWCLK: IC1.PA14, R2.2
- new net SWDIO: IC1.PA13, R1.1
- new net TFT_CLK: J10.1, SV2.17
- new net TFT_CS: IC1.PB12, J10.4, R10.1, SV1.18, SV2.14
- new net TFT_DC: IC1.PC6, J10.5, SV1.17, SV2.13
- new net TFT_MISO: IC1.PB14, J10.2, SV2.16
- new net TFT_MOSI: IC1.PB15, J10.3, SV2.15
- new net TFT_RST: IC1.PC7
- new net TFT_SCK: IC1.PB13
- new net VDDA: C7.1, C8.1, IC1.VDDA/VREF+, IC3.VO
- new net V_BASE: IC4.BASE, Q1.B
- new net V_FB: IC4.VFB, R3.1, R4.2
- new net WR: SV1.16
- new net X+: IC1.PB1, J11.2, SV1.12, SV2.9
- new net X-: IC1.PC4, J11.4, SV1.10, SV2.7
- new net Y+: IC1.PB0, J11.1, SV1.11, SV2.10
- new net Y-: IC1.PC5, J11.3, SV1.9, SV2.8
- new net ~RST: SV1.14, SV2.12
- net GND: now also C10.2, C11.2, C12.2, C13.2, C14.2, C15.2, C16.2, C17.1, C6.2, C7.2, C8.2, C9.1, IC1.VSSA/VREF-, IC1.VSS_1, IC1.VSS_2, IC1.VSS_3, IC1.VSS_4, IC3.GND, IC3.VINH, IC4.AGND, IC4.XI, J4.1, J4.2, J5.3, J6.4, J7.3, J8.3, R2.1, R4.1, R5.1, R6.1, SJ2.2, SV1.20, SV2.20
- net V_BATT: now also C10.1, C6.1, IC3.V1
Other:
- note added: "ADC Debug"
- note added: "AVDD will regulate to ~2.75V."
- note added: "Analog Voltage Regulation"
- note added: "Analog Voltage Regulator"
- note added: "Backlight Debug"
- note added: "Button / ADC Header"
- note added: "D7-D0 unused"
- note added: "Design Notes: (1) X0 = NC, XI = 0 for internal crystal oscillator (2) AVDD generated by HX711 as shown on pg. 4 of datasheet: V_avdd = V_bg * (1 + R1/R2) // incorrect in datasheet MUST be at least 0.1V less than VSUP (3) SDATA and SD_CLK go directly to microntroller input header (4) RATE = 0 means a 10Hz sampling frequency. 1 for 80 Hz. Both pull-up and pull down resistor pads will exist. (5) DVD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"
- note added: "Digital Voltage Regulator"
- note added: "Don't forget pull-up resistors on the I2C SCL and SDA lines (they're open drain)."
- note added: "HX711 Decoupling"
- note added: "HX711 Load Cell IC Biasing"
- note added: "HX711 PCB (Needs Scoring)"
- note added: "HX711 to Load Cell"
- note added: "HX711 to MCU"
- note added: "Header 1"
- note added: "Header 3"
- note added: "LHS (8-Bit Parallel Header)"
- note added: "MCU to HX711"
- note added: "MCU to MAX7219"
- note added: "NOTE: Put on silkscreen the way to close these solder jumpers (high = 80Hz sampling, low = 10 Hz sampling)"
- note added: "RHS (Serial Header)"
- note added: "STM32F401 Microcontroller"
- note added: "SWDIO - 100k pull up (ARM) SWCLK - 100k pull down (ARM)"
- note added: "Scope Probe GND Connector"
- note added: "Scope Probe VDD Connector"
- note added: "TFT LCD 2.8" Adafruit RT Touchscreen"
- note added: "TFT SPI Debug"
- note added: "TODO: Add 3-pin or 4-pin SWD header (maybe not VCC)"
- note added: "TODO: Add EEPROM Circuit Here!"
- note added: "TODO: Add MCP73831 Charging Circuit"
- note added: "TODO: Add biasing circuitry between CH+ and CH- (see datasheet)"
- note added: "TODO: Add external crystal"
- note added: "The circuit contained above is the circuit given on the HX711 development board Joe gave to me. AVDD: Positive excitation (+2.75V regulated) GND : Negative Excitation (GND) CH+: Channel A positive differential (load cell green) CH-: Channel A negative differential (load cell white) GPIO "Bit-Banged" Pins: (1) HX_SDA (2) HX_CLOCK"
- note added: "Useful Headers"
- note added: "V_FB will be internally regulated to 1.25V by the HX711 IC."
- note removed: "TIM4 CH4: PB9 (Load Cell SDCLK) Generic GPIO: PB8 (Load Cell SDATA) SPI1 SCK: ??? (TFT LCD) SPI1 MOSI: ??? (TFT LCD) SPI1 MISO: ??? (TFT LCD) SPI1 NSS: ??? (TFT LCD) I2Cx SCLK: ??? I2Cx SDA: ??? SPI2 SCK: ??? (SS Display) SPI2 MOSI: ??? (SS Display) SPI2 NSS: ??? (SS Display) SWDIO: PA13? SWCLK: PA14? SWnRST?: PA15? === Extra Pins (Redundant) === ADC0_CH0: ??? SPI4_SCK: SPI4_MOSI:"
- moved on the sheet: C1, C2, C3, C4, C5, IC1, IC2
