File: pcb/micro-board.brd (EAGLE design)
At the start: 127 x 76.2 mm, 110 parts, among them IC1 STM32F401RET6U, IC2 LDS3985M33R, IC3 LDS3985M33R, IC4 HX711, IC5 TLV2462IP, J12 B2B-PH-K-S_LF__SN_, J14 Digital LED, J15 Analog LED, J16 HX711 LED, J18 DC Power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

Commit message: Updated the micro-board.brd file with power supply + basic polygons
Parts:
- J14: value Digital LED -> 3V3 LED
- J15: value Analog LED -> VDDA LED
- LED3: value Blue -> VDD
- LED4: value Blue -> VDDA
- R15: value 330 -> 470
- moved R20 104.1 mm to (31.8, 58.4), flipped to the bottom, turned to 90 degrees
- moved C24 84.4 mm to (20.3, 71.1), turned to 270 degrees
- moved R24 73.7 mm to (47.0, 61.5), turned to 90 degrees
- moved R25 72.4 mm to (41.9, 61.6), turned to 90 degrees
- moved U1 61.7 mm to (16.5, 71.1), turned to 270 degrees
- moved R23 55.3 mm to (31.8, 54.6), flipped to the bottom, turned to 90 degrees
- moved R22 38.4 mm to (19.3, 60.8), flipped to the bottom, turned to 90 degrees
- moved R21 34.6 mm to (19.3, 64.4), flipped to the bottom, turned to 90 degrees
- moved LED2 28.2 mm to (7.62, 62.2), turned to 270 degrees
- moved R16 24.7 mm to (10.7, 63.2), turned to 180 degrees
- moved J18 19.1 mm to (29.2, 72.4), turned to 270 degrees
- moved C22 15.5 mm to (24.1, 71.1), turned to 90 degrees
- moved LED1 14.9 mm to (3.81, 62.2)
- moved R15 14.1 mm to (5.71, 65.2)
- moved IC2 10.9 mm to (47.0, 71.1)
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Routing:
- net STAT: track 0.00 -> 20.6 mm, vias 0 -> 1
- net N$4: track 0.00 -> 18.8 mm
- net N$6: track 0.00 -> 15.5 mm
- net 5V: track 0.00 -> 11.9 mm, vias 0 -> 1
- net V_LO: track 0.00 -> 4.66 mm
- net V_HI: track 0.00 -> 4.28 mm
- net GND: track 9.46 -> 13.3 mm, vias 0 -> 2
- net N$2: track 0.00 -> 2.48 mm
- net ANA_LED: track 0.00 -> 2.32 mm
- net N$5: track 0.00 -> 2.26 mm
- net N$9: track 0.00 -> 1.83 mm
- added copper zone on layer 1, net 5V
- added copper zone on layer 1, net GND
- added copper zone on layer 1, net V_BATT

Commit message: Updated power supply, decoupling, analog and digital GND
Parts:
- moved C2 103.5 mm to (28.6, 64.9), turned to 270 degrees
- moved C3 100.0 mm to (26.9, 64.9), turned to 270 degrees
- moved R35 93.0 mm to (24.4, 60.7), turned to 180 degrees
- moved R17 90.3 mm to (19.4, 73.7)
- moved R34 89.0 mm to (24.3, 65.3), turned to 180 degrees
- moved R18 87.8 mm to (22.1, 71.1), flipped to the bottom, turned to 270 degrees
- moved R19 84.9 mm to (14.9, 74.0), flipped to the bottom, turned to 180 degrees
- moved IC3 69.6 mm to (20.3, 59.7)
- moved C7 65.5 mm to (41.7, 36.8), turned to 90 degrees
- moved C9 52.1 mm to (24.4, 58.7), turned to 180 degrees
- moved C10 46.5 mm to (14.6, 59.7), turned to 270 degrees
- moved C6 43.3 mm to (16.1, 59.7), turned to 270 degrees
- moved C4 42.4 mm to (24.3, 63.8), turned to 180 degrees
- moved C8 42.2 mm to (26.9, 59.6), turned to 270 degrees
- moved C1 40.0 mm to (16.1, 62.5)
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Routing:
- net GND: track 13.3 -> 57.4 mm, vias 2 -> 7
- net STAT: track 20.6 -> 46.5 mm
- net 5V: track 11.9 -> 37.0 mm
- net V_BATT: track 0.00 -> 20.4 mm
- net N$6: track 15.5 -> 21.7 mm
- net N$4: track 18.8 -> 24.0 mm
- net VDDA: track 0.00 -> 4.42 mm
- net 3.3V: track 9.70 -> 13.4 mm
- net V_LO: track 4.66 -> 7.16 mm
- net N$19: track 0.00 -> 2.02 mm
- net N$15: track 0.00 -> 1.99 mm
- net N$1: track 0.00 -> 1.99 mm
- net N$7: track 0.00 -> 1.93 mm
- net N$3: track 0.00 -> 1.86 mm
- added copper zone on layer 1, net 3V3
Other:
- board text added: "Analog Side"
- board text added: "Digital Side"

Commit message: Finished simplistic EEPROM routing on back of main board
Parts:
- added R36, R37: 1k, LinnesLab-Passives:R0603
- added U2: BR24S64FJ-WE2, I2C-EEPROM:SOIC8
Connections:
- net 3.3V: now also R36.1, R37.1, U2.8
- net GND: now also U2.1, U2.2, U2.3, U2.4, U2.7
- net MEM_SCL: now also R36.2, U2.6
- net MEM_SDA: now also R37.2, U2.5
Routing:
- net MEM_SDA: track 0.00 -> 17.1 mm, vias 0 -> 3
- net MEM_SCL: track 0.00 -> 15.9 mm, vias 0 -> 1
- net GND: track 57.4 -> 66.5 mm
- net 3.3V: track 13.4 -> 14.4 mm, vias 0 -> 1
Changed lines of the file:
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@@
 <setting verticaltext="up"/>
 </settings>
-<grid distance="50" unitdist="mil" unit="mil" style="lines" multiple="1" display="yes" altdistance="5" altunitdist="mil" altunit="mil"/>
+<grid distance="10" unitdist="mil" unit="mil" style="lines" multiple="1" display="yes" altdistance="5" altunitdist="mil" altunit="mil"/>
 <layers>
 <layer number="1" name="Top" color="4" fill="1" visible="yes" active="yes"/>
@@
 <attribute name="VALUE" x="17.272" y="68.58" size="0.6096" layer="27" ratio="20" align="bottom-center"/>
 </element>
+<element name="U2" library="I2C-EEPROM" package="SOIC8" value="BR24S64FJ-WE2" x="53.34" y="58.42" smashed="yes" rot="MR180">
+<attribute name="NAME" x="50.673" y="60.325" size="1.27" layer="26" rot="MR270"/>
+<attribute name="VALUE" x="57.277" y="60.325" size="1.27" layer="28" rot="MR270"/>
+</element>
+<element name="R36" library="LinnesLab-Passives" package="R0603" package3d_urn="urn:adsk.eagle:package:15661944/2" value="1k" x="-85.09" y="-8.89" smashed="yes">
+<attribute name="NAME" x="-85.725" y="-8.255" size="0.7112" layer="25"/>
+<attribute name="VALUE" x="-85.725" y="-10.795" size="0.7112" layer="27"/>
+</element>
+<element name="R37" library="LinnesLab-Passives" package="R0603" package3d_urn="urn:adsk.eagle:package:15661944/2" value="1k" x="-85.09" y="-13.97" smashed="yes">
+<attribute name="NAME" x="-85.725" y="-13.335" size="0.7112" layer="25"/>
+<attribute name="VALUE" x="-85.725" y="-15.875" size="0.7112" layer="27"/>
+</element>
 </elements>
 <signals>
@@
 <vertex x="127" y="0"/>
 </polygon>
+<contactref element="U2" pad="4"/>
+<contactref element="U2" pad="3"/>
+<contactref element="U2" pad="2"/>
+<contactref element="U2" pad="1"/>
+<contactref element="U2" pad="7"/>
+<wire x1="51.435" y1="61.02" x2="52.832" y2="61.02" width="0.508" layer="16"/>
+<wire x1="52.832" y1="61.02" x2="55.245" y2="61.02" width="0.508" layer="16"/>
+<wire x1="52.705" y1="55.82" x2="52.705" y2="60.893" width="0.508" layer="16"/>
+<wire x1="52.705" y1="60.893" x2="52.832" y2="61.02" width="0.508" layer="16"/>
 <wire x1="112.395" y1="40.812" x2="111.367" y2="57.15" width="0" layer="19" extent="1-1"/>
 <wire x1="88.9" y1="53.34" x2="111.367" y2="57.15" width="0" layer="19" extent="1-1"/>
 <wire x1="78.74" y1="69.85" x2="88.9" y2="53.34" width="0" layer="19" extent="1-1"/>
-<wire x1="60.96" y1="47.752" x2="78.74" y2="69.85" width="0" layer="19" extent="1-1"/>
-<wire x1="57.277" y1="42.965" x2="60.96" y2="47.752" width="0" layer="19" extent="1-1"/>
-<wire x1="55.268" y1="42.62" x2="57.277" y2="42.965" width="0" layer="19" extent="1-1"/>
-<wire x1="46.28" y1="45.108" x2="55.268" y2="42.62" width="0" layer="19" extent="1-1"/>
-<wire x1="46.824" y1="46.863" x2="46.28" y2="45.108" width="0" layer="19" extent="1-1"/>
+<wire x1="55.245" y1="61.02" x2="78.74" y2="69.85" width="0" layer="19" extent="16-16"/>
+<wire x1="53.975" y1="61.02" x2="55.245" y2="61.02" width="0" layer="19" extent="16-16"/>
+<wire x1="52.705" y1="61.02" x2="51.435" y2="61.02" width="0" layer="19" extent="16-16"/>
+<wire x1="46.99" y1="57.162" x2="51.435" y2="61.02" width="0" layer="19" extent="1-16"/>
+<wire x1="46.824" y1="46.863" x2="46.99" y2="57.162" width="0" layer="19" extent="1-1"/>
+<wire x1="46.28" y1="45.108" x2="46.824" y2="46.863" width="0" layer="19" extent="1-1"/>
 <wire x1="43.792" y1="37.62" x2="46.28" y2="45.108" width="0" layer="19" extent="1-1"/>
 <wire x1="46.28" y1="33.632" x2="43.792" y2="37.62" width="0" layer="19" extent="1-1"/>
@@
 <wire x1="52.236" y1="31.623" x2="46.28" y2="33.632" width="0" layer="19" extent="1-1"/>
 <wire x1="52.78" y1="33.632" x2="52.236" y2="31.623" width="0" layer="19" extent="1-1"/>
-<wire x1="46.99" y1="57.162" x2="46.824" y2="46.863" width="0" layer="19" extent="1-1"/>
+<wire x1="55.268" y1="42.62" x2="46.28" y2="45.108" width="0" layer="19" extent="1-1"/>
+<wire x1="57.277" y1="42.965" x2="55.268" y2="42.62" width="0" layer="19" extent="1-1"/>
+<wire x1="60.96" y1="47.752" x2="57.277" y2="42.965" width="0" layer="19" extent="1-1"/>
 <wire x1="30.9" y1="38.227" x2="41.656" y2="37.68" width="0" layer="19" extent="1-1"/>
 <wire x1="31.75" y1="48.68" x2="30.9" y2="43.053" width="0" layer="19" extent="1-16"/>
@@
 <signal name="MEM_SCL">
 <contactref element="IC1" pad="58"/>
+<contactref element="U2" pad="6"/>
+<contactref element="R36" pad="2"/>
+<wire x1="48.78" y1="45.108" x2="48.78" y2="43.93" width="0.2032" layer="1"/>
+<wire x1="48.78" y1="43.93" x2="49.022" y2="43.688" width="0.2032" layer="1"/>
+<via x="49.022" y="43.688" extent="1-16" drill="0.35"/>
+<wire x1="49.022" y1="43.688" x2="49.276" y2="43.688" width="0.2032" layer="16"/>
+<wire x1="49.276" y1="43.688" x2="53.975" y2="48.387" width="0.2032" layer="16"/>
+<wire x1="53.975" y1="48.387" x2="53.975" y2="55.82" width="0.2032" layer="16"/>
+<wire x1="49.022" y1="43.688" x2="-84.24" y2="-8.89" width="0" layer="19" extent="1-1"/>
 </signal>
 <signal name="MEM_SDA">
 <contactref element="IC1" pad="59"/>
+<contactref element="U2" pad="5"/>
+<contactref element="R37" pad="2"/>
+<wire x1="48.28" y1="45.108" x2="48.28" y2="43.962" width="0.2032" layer="1"/>
+<wire x1="48.28" y1="43.962" x2="48.26" y2="43.942" width="0.2032" layer="1"/>
+<via x="48.26" y="43.942" extent="1-16" drill="0.35"/>
+<wire x1="48.26" y1="43.942" x2="48.768" y2="44.45" width="0.2032" layer="16"/>
+<wire x1="55.245" y1="50.546" x2="55.245" y2="55.82" width="0.2032" layer="16"/>
+<wire x1="48.768" y1="44.45" x2="48.768" y2="45.974" width="0.2032" layer="16"/>
+<via x="53.34" y="50.546" extent="1-16" drill="0.35"/>
+<wire x1="53.34" y1="50.546" x2="55.245" y2="50.546" width="0.2032" layer="1"/>
+<via x="55.245" y="50.546" extent="1-16" drill="0.35"/>
+<wire x1="48.768" y1="45.974" x2="53.34" y2="50.546" width="0.2032" layer="16"/>
+<wire x1="48.26" y1="43.942" x2="-84.24" y2="-13.97" width="0" layer="19" extent="1-1"/>
 </signal>
 <signal name="PC3">
@@
 <wire x1="25.576" y1="65.747" x2="26.924" y2="65.747" width="0.508" layer="1"/>
 <wire x1="26.924" y1="65.747" x2="28.575" y2="65.747" width="0.508" layer="1"/>
+<contactref element="U2" pad="8"/>
+<contactref element="R36" pad="1"/>
+<contactref element="R37" pad="1"/>
+<wire x1="51.435" y1="55.82" x2="50.987" y2="55.372" width="0.508" layer="16"/>
+<wire x1="50.987" y1="55.372" x2="50.546" y2="55.372" width="0.508" layer="16"/>
+<via x="50.546" y="55.372" extent="1-16" drill="0.6"/>
 <wire x1="109.855" y1="40.812" x2="111.76" y2="50.8" width="0" layer="19" extent="1-1"/>
 <wire x1="109.855" y1="35.388" x2="109.855" y2="40.812" width="0" layer="19" extent="1-1"/>
+<wire x1="88.9" y1="50.8" x2="111.76" y2="50.8" width="0" layer="19" extent="1-1"/>
 <wire x1="105.41" y1="11.43" x2="109.855" y2="35.388" width="0" layer="19" extent="1-1"/>
 <wire x1="118.11" y1="5.08" x2="105.41" y2="11.43" width="0" layer="19" extent="1-1"/>
-<wire x1="88.9" y1="50.8" x2="111.76" y2="50.8" width="0" layer="19" extent="1-1"/>
 <wire x1="68.58" y1="69.85" x2="88.9" y2="50.8" width="0" layer="19" extent="1-1"/>
 <wire x1="46.99" y1="67.31" x2="68.58" y2="69.85" width="0" layer="19" extent="1-1"/>
-<wire x1="28.575" y1="65.747" x2="46.99" y2="67.31" width="0" layer="19" extent="1-1"/>
-<wire x1="45.124" y1="46.863" x2="46.99" y2="67.31" width="0" layer="19" extent="1-1"/>
+<wire x1="51.435" y1="55.82" x2="46.99" y2="67.31" width="0" layer="19" extent="16-16"/>
+<wire x1="45.124" y1="46.863" x2="50.546" y2="55.372" width="0" layer="19" extent="1-1"/>
 <wire x1="43.792" y1="43.12" x2="45.78" y2="45.108" width="0" layer="19" extent="1-1"/>
 <wire x1="55.268" y1="43.12" x2="45.78" y2="45.108" width="0" layer="19" extent="1-1"/>
 <wire x1="53.28" y1="33.632" x2="55.268" y2="43.12" width="0" layer="19" extent="1-1"/>
 <wire x1="46.78" y1="33.632" x2="53.28" y2="33.632" width="0" layer="19" extent="1-1"/>
+<wire x1="28.575" y1="65.747" x2="46.99" y2="67.31" width="0" layer="19" extent="1-1"/>
 <wire x1="12.7" y1="7.62" x2="46.443" y2="31.623" width="0" layer="19" extent="1-1"/>
 <wire x1="-19.05" y1="67.31" x2="25.107" y2="65.278" width="0" layer="19" extent="1-1"/>
@@
 <wire x1="-42.76" y1="48.26" x2="-46.57" y2="48.26" width="0" layer="19" extent="1-1"/>
 <wire x1="-38.1" y1="72.39" x2="-42.76" y2="63.5" width="0" layer="19" extent="1-1"/>
+<wire x1="-85.94" y1="-8.89" x2="-46.57" y2="48.26" width="0" layer="19" extent="1-1"/>
+<wire x1="-85.94" y1="-13.97" x2="-85.94" y2="-8.89" width="0" layer="19" extent="1-1"/>
 </signal>
 <signal name="HX_SDA">

Commit message: Updated EEPROM Resistor Positions
Parts:
- moved R37 151.6 mm to (51.6, 51.6), flipped to the bottom, turned to 180 degrees
- moved R36 150.2 mm to (51.6, 53.3), flipped to the bottom, turned to 180 degrees
Routing:
- net 3.3V: track 14.4 -> 18.3 mm
- net MEM_SDA: track 17.1 -> 19.3 mm
- net MEM_SCL: track 15.9 -> 17.7 mm
Changed lines of the file:
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@@
 <attribute name="VALUE" x="57.277" y="60.325" size="1.27" layer="28" rot="MR270"/>
 </element>
-<element name="R36" library="LinnesLab-Passives" package="R0603" package3d_urn="urn:adsk.eagle:package:15661944/2" value="1k" x="-85.09" y="-8.89" smashed="yes">
-<attribute name="NAME" x="-85.725" y="-8.255" size="0.7112" layer="25"/>
-<attribute name="VALUE" x="-85.725" y="-10.795" size="0.7112" layer="27"/>
+<element name="R36" library="LinnesLab-Passives" package="R0603" package3d_urn="urn:adsk.eagle:package:15661944/2" value="1k" x="51.562" y="53.34" smashed="yes" rot="MR180">
+<attribute name="NAME" x="50.927" y="52.705" size="0.7112" layer="26" rot="MR180"/>
+<attribute name="VALUE" x="50.927" y="55.245" size="0.7112" layer="28" rot="MR180"/>
 </element>
-<element name="R37" library="LinnesLab-Passives" package="R0603" package3d_urn="urn:adsk.eagle:package:15661944/2" value="1k" x="-85.09" y="-13.97" smashed="yes">
-<attribute name="NAME" x="-85.725" y="-13.335" size="0.7112" layer="25"/>
-<attribute name="VALUE" x="-85.725" y="-15.875" size="0.7112" layer="27"/>
+<element name="R37" library="LinnesLab-Passives" package="R0603" package3d_urn="urn:adsk.eagle:package:15661944/2" value="1k" x="51.562" y="51.562" smashed="yes" rot="MR180">
+<attribute name="NAME" x="50.927" y="50.927" size="0.7112" layer="26" rot="MR180"/>
+<attribute name="VALUE" x="50.927" y="53.467" size="0.7112" layer="28" rot="MR180"/>
 </element>
 </elements>
@@
 <wire x1="49.022" y1="43.688" x2="49.276" y2="43.688" width="0.2032" layer="16"/>
 <wire x1="49.276" y1="43.688" x2="53.975" y2="48.387" width="0.2032" layer="16"/>
-<wire x1="53.975" y1="48.387" x2="53.975" y2="55.82" width="0.2032" layer="16"/>
-<wire x1="49.022" y1="43.688" x2="-84.24" y2="-8.89" width="0" layer="19" extent="1-1"/>
+<wire x1="53.975" y1="48.387" x2="53.975" y2="54.102" width="0.2032" layer="16"/>
+<wire x1="53.975" y1="54.102" x2="53.975" y2="55.82" width="0.2032" layer="16"/>
+<wire x1="52.412" y1="53.34" x2="53.213" y2="53.34" width="0.2032" layer="16"/>
+<wire x1="53.213" y1="53.34" x2="53.975" y2="54.102" width="0.2032" layer="16"/>
 </signal>
 <signal name="MEM_SDA">
@@
 <via x="48.26" y="43.942" extent="1-16" drill="0.35"/>
 <wire x1="48.26" y1="43.942" x2="48.768" y2="44.45" width="0.2032" layer="16"/>
-<wire x1="55.245" y1="50.546" x2="55.245" y2="55.82" width="0.2032" layer="16"/>
-<wire x1="48.768" y1="44.45" x2="48.768" y2="45.974" width="0.2032" layer="16"/>
-<via x="53.34" y="50.546" extent="1-16" drill="0.35"/>
-<wire x1="53.34" y1="50.546" x2="55.245" y2="50.546" width="0.2032" layer="1"/>
-<via x="55.245" y="50.546" extent="1-16" drill="0.35"/>
-<wire x1="48.768" y1="45.974" x2="53.34" y2="50.546" width="0.2032" layer="16"/>
-<wire x1="48.26" y1="43.942" x2="-84.24" y2="-13.97" width="0" layer="19" extent="1-1"/>
+<wire x1="48.768" y1="44.45" x2="48.768" y2="45.212" width="0.2032" layer="16"/>
+<wire x1="48.768" y1="45.212" x2="52.832" y2="49.276" width="0.2032" layer="16"/>
+<wire x1="52.412" y1="51.562" x2="52.412" y2="49.696" width="0.2032" layer="16"/>
+<wire x1="52.412" y1="49.696" x2="52.832" y2="49.276" width="0.2032" layer="16"/>
+<via x="52.832" y="49.276" extent="1-16" drill="0.35"/>
+<wire x1="52.832" y1="49.276" x2="53.848" y2="50.292" width="0.2032" layer="1"/>
+<wire x1="53.848" y1="50.292" x2="55.118" y2="50.292" width="0.2032" layer="1"/>
+<via x="55.118" y="50.292" extent="1-16" drill="0.35"/>
+<wire x1="55.245" y1="55.82" x2="55.372" y2="55.693" width="0.2032" layer="16"/>
+<wire x1="55.372" y1="55.693" x2="55.372" y2="50.546" width="0.2032" layer="16"/>
+<wire x1="55.118" y1="50.292" x2="55.372" y2="50.546" width="0.2032" layer="16"/>
 </signal>
 <signal name="PC3">
@@
 <wire x1="50.987" y1="55.372" x2="50.546" y2="55.372" width="0.508" layer="16"/>
 <via x="50.546" y="55.372" extent="1-16" drill="0.6"/>
+<wire x1="50.546" y1="55.372" x2="50.712" y2="55.206" width="0.2032" layer="16"/>
+<wire x1="50.712" y1="55.206" x2="50.712" y2="53.34" width="0.2032" layer="16"/>
+<wire x1="50.712" y1="53.34" x2="50.712" y2="51.562" width="0.2032" layer="16"/>
 <wire x1="109.855" y1="40.812" x2="111.76" y2="50.8" width="0" layer="19" extent="1-1"/>
 <wire x1="109.855" y1="35.388" x2="109.855" y2="40.812" width="0" layer="19" extent="1-1"/>
@@
 <wire x1="46.99" y1="67.31" x2="68.58" y2="69.85" width="0" layer="19" extent="1-1"/>
 <wire x1="51.435" y1="55.82" x2="46.99" y2="67.31" width="0" layer="19" extent="16-16"/>
-<wire x1="45.124" y1="46.863" x2="50.546" y2="55.372" width="0" layer="19" extent="1-1"/>
+<wire x1="45.124" y1="46.863" x2="50.712" y2="51.562" width="0" layer="19" extent="1-16"/>
 <wire x1="43.792" y1="43.12" x2="45.78" y2="45.108" width="0" layer="19" extent="1-1"/>
-<wire x1="55.268" y1="43.12" x2="45.78" y2="45.108" width="0" layer="19" extent="1-1"/>
+<wire x1="57.277" y1="44.665" x2="50.712" y2="51.562" width="0" layer="19" extent="1-16"/>
 <wire x1="53.28" y1="33.632" x2="55.268" y2="43.12" width="0" layer="19" extent="1-1"/>
 <wire x1="46.78" y1="33.632" x2="53.28" y2="33.632" width="0" layer="19" extent="1-1"/>
@@
 <wire x1="-42.76" y1="48.26" x2="-46.57" y2="48.26" width="0" layer="19" extent="1-1"/>
 <wire x1="-38.1" y1="72.39" x2="-42.76" y2="63.5" width="0" layer="19" extent="1-1"/>
-<wire x1="-85.94" y1="-8.89" x2="-46.57" y2="48.26" width="0" layer="19" extent="1-1"/>
-<wire x1="-85.94" y1="-13.97" x2="-85.94" y2="-8.89" width="0" layer="19" extent="1-1"/>
 </signal>
 <signal name="HX_SDA">

Commit message: Incremental commit of changes
Parts:
- moved C12 93.7 mm to (53.6, 29.2), flipped to the bottom, turned to 270 degrees
- moved C11 87.2 mm to (50.8, 29.2), flipped to the bottom, turned to 270 degrees
Routing:
- net N$8: track 0.00 -> 8.60 mm, vias 0 -> 1
Changed lines of the file:
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@@
 <attribute name="VALUE" x="12.7" y="60.325" size="0.7112" layer="27" rot="R270"/>
 </element>
-<element name="C11" library="LinnesLab-Passives" package="C0603" package3d_urn="urn:adsk.eagle:package:15661989/2" value="2.2uF" x="-34.29" y="48.26" smashed="yes">
-<attribute name="NAME" x="-34.925" y="48.895" size="0.7112" layer="25"/>
-<attribute name="VALUE" x="-34.925" y="46.355" size="0.7112" layer="27"/>
-</element>
-<element name="C12" library="LinnesLab-Passives" package="C0603" package3d_urn="urn:adsk.eagle:package:15661989/2" value="2.2uF" x="-38.1" y="48.26" smashed="yes">
-<attribute name="NAME" x="-38.735" y="48.895" size="0.7112" layer="25"/>
-<attribute name="VALUE" x="-38.735" y="46.355" size="0.7112" layer="27"/>
+<element name="C11" library="LinnesLab-Passives" package="C0603" package3d_urn="urn:adsk.eagle:package:15661989/2" value="2.2uF" x="50.8" y="29.21" smashed="yes" rot="MR270">
+<attribute name="NAME" x="50.165" y="29.845" size="0.7112" layer="26" rot="MR270"/>
+<attribute name="VALUE" x="52.705" y="29.845" size="0.7112" layer="28" rot="MR270"/>
+</element>
+<element name="C12" library="LinnesLab-Passives" package="C0603" package3d_urn="urn:adsk.eagle:package:15661989/2" value="2.2uF" x="53.594" y="29.21" smashed="yes" rot="MR270">
+<attribute name="NAME" x="52.959" y="29.845" size="0.7112" layer="26" rot="MR270"/>
+<attribute name="VALUE" x="55.499" y="29.845" size="0.7112" layer="28" rot="MR270"/>
 </element>
 <element name="C13" library="LinnesLab-Passives" package="C0603" package3d_urn="urn:adsk.eagle:package:15661989/2" value="10uF" x="-30.48" y="53.34" smashed="yes">
@@
 <wire x1="52.236" y1="31.623" x2="46.28" y2="33.632" width="0" layer="19" extent="1-1"/>
 <wire x1="52.78" y1="33.632" x2="52.236" y2="31.623" width="0" layer="19" extent="1-1"/>
+<wire x1="53.594" y1="28.36" x2="52.236" y2="31.623" width="0" layer="19" extent="1-16"/>
+<wire x1="50.8" y1="28.36" x2="53.594" y2="28.36" width="0" layer="19" extent="16-16"/>
 <wire x1="55.268" y1="42.62" x2="46.28" y2="45.108" width="0" layer="19" extent="1-1"/>
 <wire x1="57.277" y1="42.965" x2="55.268" y2="42.62" width="0" layer="19" extent="1-1"/>
@@
 <wire x1="-38.95" y1="53.34" x2="-41.06" y2="53.34" width="0" layer="19" extent="1-1"/>
 <wire x1="-41.06" y1="48.26" x2="-41.06" y2="53.34" width="0" layer="19" extent="1-1"/>
-<wire x1="-37.25" y1="48.26" x2="-41.06" y2="48.26" width="0" layer="19" extent="1-1"/>
-<wire x1="-33.44" y1="48.26" x2="-37.25" y2="48.26" width="0" layer="19" extent="1-1"/>
 <wire x1="-44.87" y1="48.26" x2="-41.06" y2="48.26" width="0" layer="19" extent="1-1"/>
-<wire x1="-33.44" y1="53.34" x2="-33.44" y2="48.26" width="0" layer="19" extent="1-1"/>
+<wire x1="-33.44" y1="53.34" x2="-38.95" y2="53.34" width="0" layer="19" extent="1-1"/>
 <wire x1="-29.63" y1="53.34" x2="-33.44" y2="53.34" width="0" layer="19" extent="1-1"/>
 <wire x1="-48.68" y1="58.42" x2="-41.06" y2="58.42" width="0" layer="19" extent="1-1"/>
@@
 <contactref element="C11" pad="1"/>
 <contactref element="C12" pad="1"/>
-<wire x1="-35.14" y1="48.26" x2="52.28" y2="33.632" width="0" layer="19" extent="1-1"/>
-<wire x1="-38.95" y1="48.26" x2="-35.14" y2="48.26" width="0" layer="19" extent="1-1"/>
+<wire x1="52.28" y1="33.632" x2="52.28" y2="34.754" width="0.2032" layer="1"/>
+<wire x1="52.28" y1="34.754" x2="52.324" y2="34.798" width="0.2032" layer="1"/>
+<via x="52.324" y="34.798" extent="1-16" drill="0.35"/>
+<wire x1="52.324" y1="34.798" x2="52.324" y2="31.584" width="0.2032" layer="16"/>
+<wire x1="52.324" y1="31.584" x2="50.8" y2="30.06" width="0.2032" layer="16"/>
+<wire x1="52.324" y1="31.584" x2="52.324" y2="31.33" width="0.2032" layer="16"/>
+<wire x1="52.324" y1="31.33" x2="53.594" y2="30.06" width="0.2032" layer="16"/>
 </signal>
 <signal name="X+">
@@
 <wire x1="57.277" y1="44.665" x2="50.712" y2="51.562" width="0" layer="19" extent="1-16"/>
 <wire x1="53.28" y1="33.632" x2="55.268" y2="43.12" width="0" layer="19" extent="1-1"/>
-<wire x1="46.78" y1="33.632" x2="53.28" y2="33.632" width="0" layer="19" extent="1-1"/>
+<wire x1="53.28" y1="33.632" x2="46.78" y2="33.632" width="0" layer="19" extent="1-1"/>
 <wire x1="28.575" y1="65.747" x2="46.99" y2="67.31" width="0" layer="19" extent="1-1"/>
 <wire x1="12.7" y1="7.62" x2="46.443" y2="31.623" width="0" layer="19" extent="1-1"/>
