File: pcb/micro-board.brd (EAGLE design)
At the start: 127 x 76.2 mm, 118 parts, among them IC1 STM32F401RET6U, IC2 LDS3985M33R, IC3 LDS3985M33R, IC4 HX711, IC5 TLV2462IP, J12 B2B-PH-K-S_LF__SN_, J14 3V3 LED, J15 VDDA LED, J16 HX711 LED, J18 DC Power, J3 Button / ADC Header, Q1 S8550, Q2 16MHz, U1 MCP73831.SOT23-5, U2 BR24S64FJ-WE2

Commit message: Further PCB development
Parts:
- moved C34 45.4 mm to (106.9, 41.7), turned to 90 degrees
- moved C33 39.5 mm to (108.5, 41.7), turned to 90 degrees
- moved C15 4.66 mm to (106.7, 34.0), flipped to the top, turned to 270 degrees
- moved C16 2.59 mm to (108.2, 34.0), flipped to the top, turned to 270 degrees
- moved J5 1.55 mm to (104.4, 52.3)
Routing:
- net GND: track 113.7 -> 108.2 mm, vias 16 -> 15
- net 3.3V: track 35.5 -> 33.6 mm, vias 2 -> 1
- net HXCLK: track 8.08 -> 8.96 mm
- net HXDATA: track 13.0 -> 13.9 mm

Commit message: Updated the initial revision of the PCB + PDFs of layout
Parts:
- removed C34: 10uF, LinnesLab-Passives:C0603
- removed S1: MOMENTARY-SWITCH-SPST-SMD-5.2-REDUNDANT, SparkFun-Switches:TACTILE_SWITCH_SMD_5.2MM
- added NRST: MOMENTARY-SWITCH-SPST-SMD-5.2-REDUNDANT, SparkFun-Switches:TACTILE_SWITCH_SMD_5.2MM
- added PWR: (no value), LinnesLab-Connectors:1X02
- added R40, R41, R42, R43: 20, LinnesLab-Passives:R0603
- added U$10: (no value), silkscreen:BURNING-OHIO2
- added U$9: (no value), silkscreen:BURNING-OHIO
- C29: value 0.1uF -> 10uF
- moved R4 182.2 mm to (115.7, 28.6), turned to 90 degrees
- moved R3 176.0 mm to (113.3, 28.6), turned to 270 degrees
- moved R2 118.5 mm to (61.3, 53.1), turned to 180 degrees
- moved R1 113.1 mm to (59.4, 45.5)
- moved C21 87.3 mm to (30.0, 53.8), turned to 270 degrees
- moved R14 71.2 mm to (8.64, 23.4), flipped to the bottom
- moved J4 32.8 mm to (2.54, 19.3)
- moved C29 29.8 mm to (106.9, 41.7), turned to 90 degrees
- moved Q1 18.2 mm to (108.2, 29.5), flipped to the bottom, turned to 270 degrees
- moved R9 8.48 mm to (85.6, 52.6), turned to 180 degrees
- moved U$8 7.62 mm to (104.1, 36.1)
- moved U$3 6.51 mm to (41.1, 47.0)
- moved R33 4.88 mm to (111.0, 49.8), turned to 180 degrees
- moved C20 4.80 mm to (13.7, 70.7), turned to 90 degrees
- moved J16 3.54 mm to (108.0, 58.7)
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- renumbered Q2 to X1, SJ1 to 80HZ, SJ2 to 10HZ, TFT to SPI
Connections:
- new net GND-ISO: C15.2, C16.2, C17.1, C29.2, C33.2, IC4.14, IC4.5, J5.1, J7.3, LED6.C, R27.1, R4.1
- new net VDD: C15.1, C16.1, C29.1, C33.1, IC4.1, IC4.16, J16.2, J5.4, Q1.1, R28.1, U$8.1
- new net VIN: J12.1, PWR.1
- new net X+_NC: SV1.12
- new net X-_NC: SV1.10
- new net Y+_NC: SV1.11
- new net Y-_NC: SV1.9
- new net _HXCLK: J5.3, R32.2
- new net _HXDATA: J5.2, R33.2
- new net _NC_MISO: IC1.22, R42.2
- new net _SS_CS: IC1.20, R40.2
- new net _SS_MOSI: IC1.23, R43.2
- new net _SS_SCK: IC1.21, R41.2
- net 3.3V: no longer C15.1, C16.1, C29.1, C33.1, C34.1, IC4.1, IC4.16, J16.2, J5.4, Q1.1, R14.2, R28.1, U$8.1
- net GND: now also R14.2; no longer C15.2, C16.2, C17.1, C29.2, C33.2, C34.2, IC4.14, IC4.5, J5.1, J7.3, LED6.C, R27.1, R4.1
- net HXCLK: no longer J5.3, R32.2
- net HXDATA: no longer J5.2, R33.2
- net N$17: now also NRST.3, NRST.4; no longer S1.3, S1.4
- net NC_MISO: now also R42.1; no longer IC1.22
- net NRST: now also NRST.1, NRST.2; no longer S1.1, S1.2
- net SS_CS: now also R40.1; no longer IC1.20
- net SS_MOSI: now also R43.1; no longer IC1.23
- net SS_SCK: now also R41.1; no longer IC1.21
- net V_BATT: now also PWR.2; no longer J12.1
- net X+: no longer SV1.12
- net X-: no longer SV1.10
- net Y+: no longer SV1.11
- net Y-: no longer SV1.9
Routing:
- net TFT_CS: track 61.1 -> 133.3 mm, vias 0 -> 1
- net TFT_DC: track 45.4 -> 98.1 mm, vias 0 -> 2
- net LITE: track 47.3 -> 99.4 mm, vias 1 -> 3
- net TFT_NRST: track 38.7 -> 88.4 mm, vias 0 -> 2
- net GND-ISO: track 0.00 -> 38.0 mm, vias 0 -> 4
- net SS_CS: track 34.7 -> 4.23 mm
- net _SS_CS: track 0.00 -> 28.7 mm
- net SS_SCK: track 32.2 -> 4.23 mm
- net _SS_SCK: track 0.00 -> 27.4 mm
- net NC_MISO: track 31.4 -> 4.23 mm
- net SS_MOSI: track 30.6 -> 4.23 mm
- net _NC_MISO: track 0.00 -> 25.7 mm
- net _SS_MOSI: track 0.00 -> 24.8 mm
- net PB3: track 0.00 -> 20.3 mm
- net PB4: track 0.00 -> 18.4 mm
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- added copper zone on layer 16, net GND-ISO
- added copper zone on layer 1, net VDD
Other:
- outline, holes or cut-outs redrawn
- board text added: "+3.3V"
- board text added: "16MHz"
- board text added: "3.3V"
- board text added: "3Vo"
- board text added: "A+"
- board text added: "A-"
- board text added: "BUTTONS / ADC"
- board text added: "CLK"
- board text added: "DATA"
- board text added: "DT"
- board text added: "E+"
- board text added: "E-"
- board text added: "HX711"
- board text added: "IM0"
- board text added: "IM1"
- board text added: "IM2"
- board text added: "IM3"
- board text added: "LITE"
- board text added: "NC_D0"
- board text added: "NC_D1"
- board text added: "NC_D2"
- board text added: "NC_D3"
- board text added: "NC_D4"
- board text added: "NC_D5"
- board text added: "NC_D6"
- board text added: "NC_D7"
- board text added: "NC_RD"
- board text added: "NC_WR"
- board text added: "NC_X+"
- board text added: "NC_X-"
- board text added: "NC_Y+"
- board text added: "NC_Y-"
- board text added: "OLED"
- board text added: "PA10"
- board text added: "PA11"
- board text added: "PA12"
- board text added: "PA9"
- board text added: "PB3"
- board text added: "PB4"
- board text added: "PB5"
- board text added: "PNP"
- board text added: "RATE"
- board text added: "RT"
- board text added: "SD_DET"
- board text added: "SD_NSS"
- board text added: "SPI TFT Header"
- board text added: "SS DISPLAY"
- board text added: "SWCLK"
- board text added: "SWDIO"
- board text added: "TO LOAD CELL"
- board text added: "TP0"
- board text added: "TP1"
- board text added: "TP2"
- board text added: "TP3"
- board text added: "Team 10: Smart Ingredient Scale Jeremy Tang - Team Leader Gautam Fotedar - Systems Engineer Ben Schwartz - Software Engineer Ryan Montsma - Hardware Engineer Board Revision 1.0"
- board text added: "VDD"
- board text added: "VDDA"
- board text added: "Yellow = Charging Green = Charged"
- board text added: "~LCD_CS"
- board text added: "~RST"
- board text removed: "TODO: Determine the mounting mechanism: standoffs?"

Commit message: Updated the PCB with more silkscreen and ESD protection resistors
Parts:
- added R44, R45, R46: 20, LinnesLab-Passives:R0603
- J3: value Button / ADC Header -> (none); device LinnesLab-Connectors:1X04 -> LinnesLab-Connectors:1X06_LOCK
- moved J9 2.54 mm to (2.54, 53.8)
- moved J3 1.67 mm to (17.3, 5.33)
Connections:
- new net N$20: J13.3, R45.1
- new net N$21: J13.4, R46.1
- new net N$8: J13.2, R44.1
- net 3.3V: now also J3.6
- net GND: now also J3.1
- net OLED_MOSI: now also R44.2; no longer J13.2
- net OLED_NSS: now also R45.2; no longer J13.3
- net OLED_SCK: now also R46.2; no longer J13.4
- net PC0: now also J3.5; no longer J3.4
- net PC1: now also J3.4; no longer J3.3
- net PC2: now also J3.3; no longer J3.2
- net PC3: now also J3.2; no longer J3.1
Routing:
- net OLED_MOSI: track 40.4 -> 36.6 mm
- net OLED_NSS: track 37.2 -> 34.0 mm
- net N$8: track 0.00 -> 2.45 mm
- net N$21: track 0.00 -> 2.45 mm
- net N$20: track 0.00 -> 2.45 mm
- net OLED_SCK: track 38.3 -> 35.9 mm
- net PC2: track 44.5 -> 43.9 mm
- net PC1: track 44.3 -> 44.4 mm, vias 0 -> 2
Other:
- board text added: "AMP"
- board text added: "OP"
