File: pcb/footprints.sch (EAGLE design)
At the start: 11 parts, among them IC1 HX711, IC2 STM32F401RET6U, IC3 LDS3985M33R, IC4 LMC555CN_NOPB, IC5 M95640-RMN6P, U1 MCP73831.SOT23-5

Commit message: Updated the PCB Schematic: 80% complete. Added PCB reference.
Parts:
- added IC6: TLV2462IP, SamacSys_Parts:TLV2462IP
- added J1: (no value), LinnesLab-Connectors:CONN_02
- added J2: (no value), LinnesLab-Connectors:CONN_04
- added LIPO1: (no value), LinnesLab-Connectors:JST_2MM_MALE
- added S1: EG1270, SamacSys_Parts:EG1270
- SV1: device con-lstb:MA20-1 -> con-lsta:FE20-1
Changed lines of the file:
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@@
 <layers>
 <layer number="1" name="Top" color="4" fill="1" visible="no" active="no"/>
+<layer number="2" name="Route2" color="1" fill="3" visible="no" active="no"/>
+<layer number="3" name="Route3" color="4" fill="3" visible="no" active="no"/>
+<layer number="4" name="Route4" color="1" fill="4" visible="no" active="no"/>
+<layer number="5" name="Route5" color="4" fill="4" visible="no" active="no"/>
+<layer number="6" name="Route6" color="1" fill="8" visible="no" active="no"/>
+<layer number="7" name="Route7" color="4" fill="8" visible="no" active="no"/>
+<layer number="8" name="Route8" color="1" fill="2" visible="no" active="no"/>
+<layer number="9" name="Route9" color="4" fill="2" visible="no" active="no"/>
+<layer number="10" name="Route10" color="1" fill="7" visible="no" active="no"/>
+<layer number="11" name="Route11" color="4" fill="7" visible="no" active="no"/>
+<layer number="12" name="Route12" color="1" fill="5" visible="no" active="no"/>
+<layer number="13" name="Route13" color="4" fill="5" visible="no" active="no"/>
+<layer number="14" name="Route14" color="1" fill="6" visible="no" active="no"/>
+<layer number="15" name="Route15" color="4" fill="6" visible="no" active="no"/>
 <layer number="16" name="Bottom" color="1" fill="1" visible="no" active="no"/>
 <layer number="17" name="Pads" color="2" fill="1" visible="no" active="no"/>
@@
 <part name="R1" library="LinnesLab-Passives" deviceset="RESISTOR" device="0603" package3d_urn="urn:adsk.eagle:package:15661944/2"/>
 <part name="C1" library="LinnesLab-Passives" deviceset="CAPACITOR" device="0603" package3d_urn="urn:adsk.eagle:package:15661989/2"/>
-<part name="SV1" library="con-lstb" library_urn="urn:adsk.eagle:library:162" deviceset="MA20-1" device="" package3d_urn="urn:adsk.eagle:package:8359/1"/>
 <part name="DCJ-0303" library="con-jack" library_urn="urn:adsk.eagle:library:154" deviceset="DCJ0303" device="" package3d_urn="urn:adsk.eagle:package:7493/1"/>
+<part name="SV1" library="con-lsta" library_urn="urn:adsk.eagle:library:161" deviceset="FE20-1" device="" package3d_urn="urn:adsk.eagle:package:8196/1"/>
+<part name="IC6" library="SamacSys_Parts" deviceset="TLV2462IP" device=""/>
+<part name="LIPO1" library="LinnesLab-Connectors" deviceset="JST_2MM_MALE" device=""/>
+<part name="J1" library="LinnesLab-Connectors" deviceset="CONN_02" device=""/>
+<part name="J2" library="LinnesLab-Connectors" deviceset="CONN_04" device=""/>
+<part name="S1" library="SamacSys_Parts" deviceset="EG1270" device=""/>
 </parts>
 <sheets>
@@
 <attribute name="VALUE" x="221.996" y="35.179" size="1.778" layer="96" rot="R180"/>
 </instance>
-<instance part="SV1" gate="1" x="218.44" y="-5.08" smashed="yes" rot="R180">
-<attribute name="VALUE" x="219.71" y="22.86" size="1.778" layer="96" rot="R180"/>
-<attribute name="NAME" x="219.71" y="-33.782" size="1.778" layer="95" rot="R180"/>
-</instance>
 <instance part="DCJ-0303" gate="G$1" x="185.42" y="-2.54" smashed="yes">
 <attribute name="NAME" x="182.88" y="1.27" size="1.778" layer="95"/>
 <attribute name="VALUE" x="182.88" y="-8.89" size="1.778" layer="96"/>
 </instance>
+<instance part="SV1" gate="G$1" x="78.74" y="-12.7" smashed="yes" rot="R270">
+<attribute name="VALUE" x="48.26" y="-11.43" size="1.778" layer="96" rot="R270"/>
+<attribute name="NAME" x="104.902" y="-11.43" size="1.778" layer="95" rot="R270"/>
+</instance>
+<instance part="IC6" gate="G$1" x="91.44" y="40.64" smashed="yes">
+<attribute name="NAME" x="115.57" y="48.26" size="1.778" layer="95" align="center-left"/>
+<attribute name="VALUE" x="115.57" y="45.72" size="1.778" layer="96" align="center-left"/>
+</instance>
+<instance part="LIPO1" gate="G$1" x="226.06" y="2.54" smashed="yes">
+<attribute name="NAME" x="223.52" y="8.382" size="1.778" layer="95"/>
+</instance>
+<instance part="J1" gate="G$1" x="162.56" y="-12.7" smashed="yes">
+<attribute name="VALUE" x="160.02" y="-17.526" size="1.778" layer="96" font="vector"/>
+<attribute name="NAME" x="160.02" y="-7.112" size="1.778" layer="95" font="vector"/>
+</instance>
+<instance part="J2" gate="G$1" x="134.62" y="-27.94" smashed="yes">
+<attribute name="VALUE" x="129.54" y="-35.306" size="1.778" layer="96" font="vector"/>
+<attribute name="NAME" x="129.54" y="-19.812" size="1.778" layer="95" font="vector"/>
+</instance>
+<instance part="S1" gate="G$1" x="180.34" y="-20.32" smashed="yes">
+<attribute name="NAME" x="199.39" y="-12.7" size="1.778" layer="95" align="center-left"/>
+<attribute name="VALUE" x="199.39" y="-15.24" size="1.778" layer="96" align="center-left"/>
+</instance>
 </instances>

Commit message: Added I2C EEPROM Footprint to both schematic and board and dimensioned appropriately
Parts:
- added U2: BR24S64FJ-WE2, I2C-EEPROM:BR24S64FJ-WE2
Changed lines of the file:
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@@
 <part name="J2" library="LinnesLab-Connectors" deviceset="CONN_04" device=""/>
 <part name="S1" library="SamacSys_Parts" deviceset="EG1270" device=""/>
+<part name="U2" library="I2C-EEPROM" deviceset="BR24S64FJ-WE2" device=""/>
 </parts>
 <sheets>
@@
 <attribute name="VALUE" x="199.39" y="-15.24" size="1.778" layer="96" align="center-left"/>
 </instance>
+<instance part="U2" gate="G$1" x="76.2" y="25.4" smashed="yes">
+<attribute name="NAME" x="45.72" y="40.64" size="2.1844" layer="95"/>
+<attribute name="VALUE" x="45.72" y="20.32" size="2.1844" layer="96"/>
+</instance>
 </instances>

Commit message: Updated the initial revision of the PCB + PDFs of layout
Parts:
- removed LIPO1: (no value), LinnesLab-Connectors:JST_2MM_MALE
- added Q1: S8550, SamacSys_Parts:S8550
Changed lines of the file:
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@@
 <part name="SV1" library="con-lsta" library_urn="urn:adsk.eagle:library:161" deviceset="FE20-1" device="" package3d_urn="urn:adsk.eagle:package:8196/1"/>
 <part name="IC6" library="SamacSys_Parts" deviceset="TLV2462IP" device=""/>
-<part name="LIPO1" library="LinnesLab-Connectors" deviceset="JST_2MM_MALE" device=""/>
 <part name="J1" library="LinnesLab-Connectors" deviceset="CONN_02" device=""/>
 <part name="J2" library="LinnesLab-Connectors" deviceset="CONN_04" device=""/>
 <part name="S1" library="SamacSys_Parts" deviceset="EG1270" device=""/>
 <part name="U2" library="I2C-EEPROM" deviceset="BR24S64FJ-WE2" device=""/>
+<part name="Q1" library="SamacSys_Parts" deviceset="S8550" device=""/>
 </parts>
 <sheets>
@@
 <attribute name="VALUE" x="115.57" y="45.72" size="1.778" layer="96" align="center-left"/>
 </instance>
-<instance part="LIPO1" gate="G$1" x="226.06" y="2.54" smashed="yes">
-<attribute name="NAME" x="223.52" y="8.382" size="1.778" layer="95"/>
-</instance>
 <instance part="J1" gate="G$1" x="162.56" y="-12.7" smashed="yes">
 <attribute name="VALUE" x="160.02" y="-17.526" size="1.778" layer="96" font="vector"/>
@@
 <attribute name="VALUE" x="45.72" y="20.32" size="2.1844" layer="96"/>
 </instance>
+<instance part="Q1" gate="G$1" x="114.3" y="73.66" smashed="yes" rot="R180">
+<attribute name="NAME" x="100.33" y="72.39" size="1.778" layer="95" rot="R180" align="center-left"/>
+<attribute name="VALUE" x="100.33" y="74.93" size="1.778" layer="96" rot="R180" align="center-left"/>
+</instance>
 </instances>
